File: MACH3_interfaz.kicad_pcb (KiCad board)
At the start: 2 copper layers, 17 parts, among them J4 Screw_Terminal_01x13, J5 B4B-XH-A_LF__SN_, J6 B4B-XH-A_LF__SN_, J7 B4B-XH-A_LF__SN_, J8 B4B-XH-A_LF__SN_, J9 B4B-XH-A_LF__SN_, Q1 2N7002, Q2 MMBT2222ALT3G, U1 74HC245, U10 PC817, U2 74HC245, U3 PC817, U4 PC817, U5 PC817, U6 PC817, U7 PC817

Commit message: Listo para revison de esquematico
Parts:
- added C1: 220uF, Capacitor_THT:CP_Radial_D6.3mm_P2.50mm, F.Cu at (119.2, 27.0)
- added C2: 100nF, Capacitor_SMD:C_0805_2012Metric_Pad1.18x1.45mm_HandSolder, F.Cu at (69.3, 46.1)
- added C3: 100nF, Capacitor_SMD:C_0805_2012Metric_Pad1.18x1.45mm_HandSolder, F.Cu at (171.0, 105.0)
- added C4: 220uF, Capacitor_THT:CP_Radial_D6.3mm_P2.50mm, F.Cu at (75.1, 40.7)
- added C5: 4.7uF, Capacitor_THT:CP_Radial_D5.0mm_P2.00mm, F.Cu at (92.0, 33.0)
- added C6: 220uF, Capacitor_THT:CP_Radial_D8.0mm_P3.80mm, F.Cu at (203.0, 104.0)
- added C7: 100nF, Capacitor_SMD:C_0805_2012Metric_Pad1.18x1.45mm_HandSolder, F.Cu at (196.0, 127.0)
- added D1: LED_Small, LED_SMD:LED_0805_2012Metric_Pad1.15x1.40mm_HandSolder, F.Cu at (181.0, 83.0)
- added D2: LED_Small, LED_SMD:LED_0805_2012Metric_Pad1.15x1.40mm_HandSolder, F.Cu at (87.5, 45.1)
- added D3: M7, Diode_SMD:D_SMA_Handsoldering, F.Cu at (184.5, 126.0)
- added D4: LED, LED_SMD:LED_0805_2012Metric_Pad1.15x1.40mm_HandSolder, F.Cu at (159.0, 51.0)
- added FID1: Fiducial, Fiducial:Fiducial_1mm_Mask3mm, F.Cu at (104.0, 126.0)
- added FID2: Fiducial, Fiducial:Fiducial_1mm_Mask3mm, F.Cu at (184.0, 88.0)
- added H1: MountingHole, MountingHole:MountingHole_3.2mm_M3, F.Cu at (104.0, 79.0)
- added H2: MountingHole, MountingHole:MountingHole_3.2mm_M3, F.Cu at (186.0, 79.0)
- added H3: MountingHole, MountingHole:MountingHole_3.2mm_M3, F.Cu at (186.0, 134.0)
- added H4: MountingHole, MountingHole:MountingHole_3.2mm_M3, F.Cu at (104.0, 134.0)
- added J1: USB_B_Micro, Connector_USB:USB_Micro-B_Amphenol_10118194_Horizontal, F.Cu at (175.0, 78.0)
- added J11: Screw_Terminal_01x06, TerminalBlock_Phoenix:TerminalBlock_Phoenix_MKDS-1,5-6_1x06_P5.00mm_Horizontal, F.Cu at (184.0, 121.0)
- added J2: DB25_Male_MountingHoles, Connector_Dsub:DSUB-25_Male_Horizontal_P2.77x2.84mm_EdgePinOffset4.94mm_Housed_MountingHolesOffset7.48mm, F.Cu at (157.9, 82.8)
- added J3: Screw_Terminal_01x06, TerminalBlock_Phoenix:TerminalBlock_Phoenix_MKDS-1,5-6_1x06_P5.00mm_Horizontal, F.Cu at (105.0, 93.0)
- added JP1: Jumper, TestPoint:TestPoint_2Pads_Pitch2.54mm_Drill0.8mm, F.Cu at (62.5, 46.0)
- added R1: 2k2, Resistor_SMD:R_0805_2012Metric_Pad1.20x1.40mm_HandSolder, F.Cu at (178.0, 84.0)
- added R10: 10k, Resistor_SMD:R_0805_2012Metric_Pad1.20x1.40mm_HandSolder, F.Cu at (125.0, 113.0)
- added R11: 1k, Resistor_SMD:R_0805_2012Metric_Pad1.20x1.40mm_HandSolder, F.Cu at (112.0, 114.0)
- added R12: 2k2, Resistor_SMD:R_0805_2012Metric_Pad1.20x1.40mm_HandSolder, F.Cu at (203.0, 120.0)
- added R13: 300, Resistor_SMD:R_0805_2012Metric_Pad1.20x1.40mm_HandSolder, F.Cu at (102.2, 38.2)
- added R14: 1k, Resistor_SMD:R_0805_2012Metric_Pad1.20x1.40mm_HandSolder, F.Cu at (137.0, 40.0)
- added R15: 12k, Resistor_SMD:R_0805_2012Metric_Pad1.20x1.40mm_HandSolder, F.Cu at (125.9, 44.8)
- added R16: 510, Resistor_SMD:R_0805_2012Metric_Pad1.20x1.40mm_HandSolder, F.Cu at (97.9, 44.8)
- added R17: 300, Resistor_SMD:R_0805_2012Metric_Pad1.20x1.40mm_HandSolder, F.Cu at (111.6, 45.1)
- added R18: 4k7, Resistor_SMD:R_0805_2012Metric_Pad1.20x1.40mm_HandSolder, F.Cu at (121.1, 45.0)
- added R19: 1k8, Resistor_SMD:R_0805_2012Metric_Pad1.20x1.40mm_HandSolder, F.Cu at (160.0, 107.0)
- added R2: 1k, Resistor_SMD:R_0805_2012Metric_Pad1.20x1.40mm_HandSolder, F.Cu at (112.0, 94.0)
- added R20: 510, Resistor_SMD:R_0805_2012Metric_Pad1.20x1.40mm_HandSolder, F.Cu at (149.0, 114.0)
- added R21: 2k2, Resistor_SMD:R_0805_2012Metric_Pad1.20x1.40mm_HandSolder, F.Cu at (102.0, 33.0)
- added R22: 2k2, Resistor_SMD:R_0805_2012Metric_Pad1.20x1.40mm_HandSolder, F.Cu at (116.4, 45.1)
- added R3: 1k, Resistor_SMD:R_0805_2012Metric_Pad1.20x1.40mm_HandSolder, F.Cu at (112.0, 99.0)
- added R4: 1k, Resistor_SMD:R_0805_2012Metric_Pad1.20x1.40mm_HandSolder, F.Cu at (112.0, 104.0)
- added R5: 10k, Resistor_SMD:R_0805_2012Metric_Pad1.20x1.40mm_HandSolder, F.Cu at (125.0, 89.0)
- added R6: 10k, Resistor_SMD:R_0805_2012Metric_Pad1.20x1.40mm_HandSolder, F.Cu at (125.0, 95.0)
- added R7: 10k, Resistor_SMD:R_0805_2012Metric_Pad1.20x1.40mm_HandSolder, F.Cu at (125.0, 101.0)
- added R8: 10k, Resistor_SMD:R_0805_2012Metric_Pad1.20x1.40mm_HandSolder, F.Cu at (125.0, 107.0)
- added R9: 1k, Resistor_SMD:R_0805_2012Metric_Pad1.20x1.40mm_HandSolder, F.Cu at (112.0, 109.0)
- added RN1: R_Pack04, Resistor_SMD:R_Array_Convex_4x1206, F.Cu at (135.0, 89.5)
- added RN2: R_Pack04, Resistor_SMD:R_Array_Convex_4x1206, F.Cu at (141.0, 89.5)
- added RN3: R_Pack04, Resistor_SMD:R_Array_Convex_4x1206, F.Cu at (155.0, 89.5)
- added U8: LM317MABDTG, Package_TO_SOT_SMD:TO-252-3_TabPin2, F.Cu at (167.9, 110.0)
- added U9: LM358, Package_SO:SOIC-8_3.9x4.9mm_P1.27mm, F.Cu at (169.5, 119.4)
- U1, U2: footprint Package_DIP:DIP-20_W7.62mm_LongPads -> Package_SO:SO-20_12.8x7.5mm_P1.27mm
- moved U2 142.5 mm to (152.6, 99.4), turned to 90 degrees
- moved Q1 141.1 mm to (159.0, 121.0)
- moved Q2 138.1 mm to (151.0, 121.0)
- moved J4 137.2 mm to (115.0, 133.0)
- moved J9 136.5 mm to (162.0, 150.0)
- moved J8 128.3 mm to (149.0, 150.0)
- moved J7 128.1 mm to (136.0, 150.0)
- moved U1 118.8 mm to (137.0, 99.4), turned to 90 degrees
- moved RLY1 116.6 mm to (166.0, 52.0)
- moved J6 116.3 mm to (123.0, 150.0)
- moved J5 102.3 mm to (110.0, 150.0)
- moved U10 97.9 mm to (152.4, 111.5)
- moved U4 75.5 mm to (115.0, 96.0)
- moved U6 71.1 mm to (115.0, 108.0)
- moved U3 70.1 mm to (115.0, 90.0)
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Connections:
- net /V_REG renamed +10V
- net GNDD renamed GND1
- J5 pad 1: Net-(J5-Pad1) -> +5V
- J5 pad 2: Net-(J5-Pad2) -> /P2
- J5 pad 3: Net-(J5-Pad3) -> /P3
- J5 pad 4: Net-(J5-Pad4) -> /EN_1
- J6 pad 1: Net-(J6-Pad1) -> +5V
- J6 pad 2: Net-(J6-Pad2) -> /P4
- J6 pad 3: Net-(J6-Pad3) -> /P5
- J6 pad 4: Net-(J6-Pad4) -> /EN_1
- J7 pad 1: Net-(J7-Pad1) -> +5V
- J7 pad 2: Net-(J7-Pad2) -> /P6
- J7 pad 3: Net-(J7-Pad3) -> /P7
- J7 pad 4: Net-(J7-Pad4) -> /EN_2
- J8 pad 1: Net-(J8-Pad1) -> +5V
- J8 pad 2: Net-(J8-Pad2) -> /P8
- J8 pad 3: Net-(J8-Pad3) -> /P9
- J8 pad 4: Net-(J8-Pad4) -> /EN_2
- J9 pad 1: Net-(J9-Pad1) -> +5V
- J9 pad 2: Net-(J9-Pad2) -> /P16
- J9 pad 3: Net-(J9-Pad3) -> /P17
- J9 pad 4: Net-(J9-Pad4) -> /EN_2
- RLY1 pad 1: Net-(J11-Pad3) -> /RL_COM
- RLY1 pad 3: Net-(J11-Pad2) -> /RL_NA
Other:
- board outline added: 90 x 63 mm
- board text added: "Grilla: 1mm"

Commit message: Para correccion Docente Eschema, Companiero PCB
Parts:
- J4: value Screw_Terminal_01x13 -> Screw_Terminal_01x15; footprint TerminalBlock_Phoenix:TerminalBlock_Phoenix_MKDS-1,5-13_1x13_P5.00mm_Horizontal -> TerminalBlock_Phoenix:TerminalBlock_Phoenix_MKDS-1,5-15_1x15_P5.00mm_Horizontal
- moved D2 136.0 mm to (190.2, 134.1), turned to 180 degrees
- moved C4 128.4 mm to (185.0, 107.0), turned to 270 degrees
- moved C5 119.5 mm to (177.0, 117.0), turned to 270 degrees
- moved C2 117.0 mm to (180.0, 84.0), turned to 90 degrees
- moved JP1 112.1 mm to (161.0, 99.5), turned to 90 degrees
- moved R16 109.1 mm to (183.0, 113.0), turned to 180 degrees
- moved R13 95.9 mm to (168.0, 108.0), turned to 90 degrees
- moved R21 90.6 mm to (164.0, 99.0), turned to 90 degrees
- moved R15 87.4 mm to (172.0, 119.0), turned to 180 degrees
- moved R18 84.3 mm to (168.0, 115.0), turned to 180 degrees
- moved R14 83.3 mm to (171.0, 116.0), turned to 90 degrees
- moved R17 83.2 mm to (166.0, 108.0), turned to 270 degrees
- moved C1 79.4 mm to (174.0, 84.5), turned to 90 degrees
- moved R22 63.3 mm to (161.0, 90.0), turned to 270 degrees
- moved D4 44.3 mm to (164.0, 95.0), turned to 270 degrees
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Connections:
- J4 pad 1: /P1 -> /P2
- J4 pad 10: /P14 -> /P16
- J4 pad 11: /P16 -> /P17
- J4 pad 12: /P17 -> /P1
- J4 pad 2: /P2 -> /P3
- J4 pad 3: /P3 -> /P4
- J4 pad 4: /P4 -> /P5
- J4 pad 5: /P5 -> /P6
- J4 pad 6: /P6 -> /P7
- J4 pad 7: /P7 -> /P8
- J4 pad 8: /P8 -> /P9
- J4 pad 9: /P9 -> /P14
Routing:
- net +5V: track 0.00 -> 306.1 mm, vias 0 -> 2
- net +10V: track 0.00 -> 221.9 mm, vias 0 -> 1
- net GND: track 0.00 -> 116.2 mm
- net /OP15: track 0.00 -> 75.1 mm
- net /P17: track 0.00 -> 65.6 mm
- net /EN_2: track 0.00 -> 62.6 mm, vias 0 -> 1
- net /P16: track 0.00 -> 56.4 mm
- net /P8: track 0.00 -> 54.4 mm
- net /P9: track 0.00 -> 52.5 mm
- net /P1: track 0.00 -> 51.2 mm, vias 0 -> 2
- net /P2: track 0.00 -> 44.5 mm
- net /OP17: track 0.00 -> 44.2 mm, vias 0 -> 1
- net /EN_1: track 0.00 -> 43.6 mm, vias 0 -> 1
- net /P6: track 0.00 -> 42.3 mm
- net /P3: track 0.00 -> 41.9 mm
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- added copper zone on B.Cu, net GND
- added copper zone on F.Cu, net GND
- added copper zone on B.Cu, net GND1
- added copper zone on F.Cu, net GND1
Other:
- board size 90 x 63 mm -> 100 x 68 mm
- board text added: "+5V CLK CW EN"
- board text added: "+5V_USB"
- board text added: "A"
- board text added: "B"
- board text added: "CLK CW EN X P2 P3 Y P4 P5 Z P6 P7 P14 A P8 P9 B P16 P17"
- board text added: "GND"
- board text added: "Grilla: 1mm / 5mils"
- board text added: "IND. ARG."
- board text added: "JST 4P"
- board text added: "P1"
- board text added: "P10"
- board text added: "P11"
- board text added: "P12"
- board text added: "P13"
- board text added: "P14"
- board text added: "P15"
- board text added: "P16"
- board text added: "P17"
- board text added: "P17 - Relay P1 - PWM"
- board text added: "P2"
- board text added: "P3"
- board text added: "P4"
- board text added: "P5"
- board text added: "P6"
- board text added: "P7"
- board text added: "P8"
- board text added: "P9"
- board text added: "PC5V"
- board text added: "PCGND"
- board text added: "PWR_ON"
- board text added: "Rev 1.0"
- board text added: "X"
- board text added: "Y"
- board text added: "Z"
- board text removed: "Grilla: 1mm"

Commit message: Listo para revision final
Parts:
- moved D4 0.60 mm to (164.6, 95.0)
- moved R21 0.60 mm to (164.6, 99.0)
- renumbered RLY1 to K1
Connections:
- net /V_IN renamed Net-(D3-Pad2)
Other:
- board text added: "INTERFAZ LPT MACH3"
- board text added: "Manufacturing Process Capabilities: Ernesto Mayer S.A. (https://www.mayerpcb.com/) Grid: 1mm / 5mils Clearence: 0.508mm Track width: 3mm / 1mm / 0.5mm / 0.4mm Via Diameter: 0.8mm Via Hole: 0.4mm Layers: 2 (Front and Bottom) Finish: Sn/Pb Solder Mask color: Black Silkscreen color: White"
- board text removed: "Grilla: 1mm / 5mils"
